Commit message: Update joint connections and origins in URDF

File: ur10_leaphand.urdf (robot description, URDF)
Before this commit: robot ur10_leaphand, 27 links, 26 joints
Joints:
- joint connect_leaphand_joint: origin xyz=0.0 0.02 0.0 rpy=1.5708 3.14159265359 0.0 -> xyz=0.04 0.0 0.0 rpy=-1.5707963267948958919 0.0 1.5707963267948958919
- joint ur5e_connect_joint: origin xyz=0.0 0.112 0.0 rpy=0.0 0.0 0.0 -> xyz=0.0 0.0 0.0 rpy=0.0 0.0 0.0; parent wrist_3_link -> ee_link
