Commit message: Update ur5e_leaphand.urdf

File: ur5e_leaphand.urdf (robot description, URDF)
Before this commit: robot ur5e_leaphand, 26 links, 25 joints
Links:
- added link ee_link; collision box size=0.01 0.01 0.01
Joints:
- added joint ee_fixed_joint: type fixed, parent wrist_3_link, child ee_link, origin xyz=0.0 0.1 0.0 rpy=0.0 0.0 1.57079632679
- joint connect_leaphand_joint: origin xyz=0.0 0.02 0.0 rpy=1.5708 3.14159265359 0.0 -> xyz=0.04 0.0 0.0 rpy=-1.570796326794896336 0.0 1.570796326794896336
- joint ur5e_connect_joint: origin xyz=0.0 0.119 0.0 rpy=0.0 0.0 0.0 -> xyz=0.0 0.0 0.0 rpy=0.0 0.0 0.0; parent wrist_3_link -> ee_link
